File: TempController4Oven_ESP8266_WithoutLCD/TempController4Oven.kicad_pcb (KiCad board)
At the start: 2 copper layers, 110 x 70 mm, 34 parts, among them J1 Jack-DC, J10 Conn_01x01_Male, J11 Conn_01x01_Male, J2 Conn_01x03_Male, J3 Conn_01x01_Male, J4 Conn_01x01_Male, J5 Conn_01x01_Male, J6 Conn_01x01_Male, J7 Conn_01x01_Male, J8 Conn_01x01_Male, J9 Conn_01x01_Male, K1 FINDER-36.11, Q1 2SC4213, U1 NodeMCU_1.0_(ESP-12E), U2 AMS1117-3.3, U3 ESP-01v090

Commit message: Add new pcb
Parts:
- moved J8 1.46 mm to (164.1, 117.8)
- moved J5 1.45 mm to (62.8, 117.8)
- moved J11 1.45 mm to (68.3, 117.7)
Routing:
- net Net-(D1-A): track 22.0 -> 24.2 mm
- net Net-(J10-Pin_1): track 102.7 -> 103.6 mm
Other:
- outline, holes or cut-outs redrawn
