File: TempController4Oven/TempController4Oven.kicad_pcb (KiCad board)
At the start: 2 copper layers, 110 x 70 mm, 37 parts, among them J1 Jack-DC, J10 Conn_01x01_Male, J11 Conn_01x01_Male, J12 Conn_01x03_Male, J2 Conn_01x03_Male, J3 Conn_01x01_Male, J4 Conn_01x01_Male, J5 Conn_01x01_Male, J6 Conn_01x01_Male, J7 Conn_01x01_Male, J8 Conn_01x01_Male, J9 Conn_01x01_Male, K1 FINDER-36.11, Q1 2SC4213, U1 STM8S003F3P, U2 AMS1117-3.3

Commit message: modifications
Parts:
- C1, C5, C6, C7: value C_Small -> 0.1uF
- C2: value C_Small -> 0.1uF/25V
- C3: value C_Polarized_Small -> 10uF
- C4: value C_Polarized_Small -> 22uF
- R1, R7: value R_Small_US -> 1.2K
- R2: value R_Small_US -> 20
- R3: value R_Small_US -> 10K
- R4: value R_Small_US -> 200
- R5: value R_Small_US -> 4.7K
- R6: value R_Small_US -> 1K
- R8: value R_Small_US -> 3.6K
- moved J2 104.9 mm to (167.8, 75.1), turned to 0 degrees
- moved J1 104.8 mm to (167.7, 85.4)
- moved J12 16.2 mm to (148.4, 89.0), turned to 90 degrees
Connections:
- net /GPIO0 renamed /LCD_EN
- net /GPIO1 renamed /LCD_RS
- net /GPIO2 renamed /LCD_D0
- net /GPIO3 renamed /LCD_D1
- net /GPIO4 renamed /LCD_D2
- net /GPIO5 renamed /LCD_D3
- net /GPIO6 renamed /GP_RELAY
- net /GPIO7 renamed /SEN_TEMP
Routing:
- net /SWIM: track 30.5 -> 11.2 mm, vias 2 -> 1
- net +5VD: track 182.7 -> 169.2 mm
- net +12V: track 95.3 -> 94.7 mm

Commit message: add modification
Parts:
- moved J4 51.5 mm to (114.2, 108.7)
- moved J7 51.5 mm to (120.0, 108.5)
- moved J3 51.1 mm to (114.1, 100.6)
- moved J9 51.1 mm to (119.7, 100.6)
- moved J11 48.5 mm to (116.3, 118.9)
- moved J5 44.8 mm to (107.5, 115.4)
- moved REF** 41.8 mm to (106.8, 123.8)
- moved REF** 41.8 mm to (106.8, 63.8)
- moved J2 10.1 mm to (167.8, 85.3), turned to 180 degrees
- moved J1 9.56 mm to (167.8, 75.9), turned to 180 degrees
- moved D1 5.79 mm to (118.9, 88.9), turned to 0 degrees
- moved J8 3.00 mm to (164.0, 114.9)
- moved R4 2.88 mm to (114.7, 68.1)
- moved J10 2.73 mm to (164.1, 107.6)
Connections:
- U1 pad 15: /LCD_EN -> /LCD_RS
- U1 pad 16: /LCD_RS -> /LCD_EN
- U1 pad 19: /LCD_D0 -> /LCD_D1
- U1 pad 20: /LCD_D1 -> /LCD_D0
Routing:
- net /SEN_TEMP: track 114.9 -> 30.4 mm, vias 2 -> 1
- net +12V: track 94.7 -> 28.1 mm, vias 1 -> 0
- net Net-(J10-Pin_1): track 101.2 -> 50.3 mm
- net +5VD: track 169.2 -> 127.4 mm, vias 7 -> 6
- net Earth_Protective: track 101.4 -> 59.6 mm
- net Net-(J3-Pin_1): track 59.6 -> 33.6 mm
- net Net-(D1-A): track 13.7 -> 26.6 mm, vias 1 -> 2
- net /LCD_D0: track 39.2 -> 34.9 mm
- net /LCD_EN: track 34.5 -> 30.5 mm, vias 1 -> 0
- net Net-(DS1-LED(+)): track 9.31 -> 6.32 mm
- net /LCD_RS: track 30.4 -> 29.5 mm
- net /LCD_D2: track 49.7 -> 50.6 mm
- net Net-(J6-Pin_1): track 40.9 -> 40.2 mm
- net /SWIM: track 11.2 -> 10.5 mm
- net GND: vias 247 -> 103
Other:
- board size 110 x 70 mm -> 68.8 x 70 mm
