File: TempController4Oven/TempController4Oven.kicad_sch (KiCad schematic)
At the start: 33 parts, among them J1 Jack-DC, J10 Conn_01x01_Male, J11 Conn_01x01_Male, J12 Conn_01x03_Male, J2 Conn_01x03_Male, J3 Conn_01x01_Male, J4 Conn_01x01_Male, J5 Conn_01x01_Male, J6 Conn_01x01_Male, J7 Conn_01x01_Male, J8 Conn_01x01_Male, J9 Conn_01x01_Male, K1 FINDER-36.11, Q1 2SC4213, U1 STM8S003F3P, U2 AMS1117-3.3

Commit message: modifications
Parts:
- C1, C5, C6, C7: value C_Small -> 0.1uF
- C2: value C_Small -> 0.1uF/25V
- C3: value C_Polarized_Small -> 10uF
- C4: value C_Polarized_Small -> 22uF
- R1, R7: value R_Small_US -> 1.2K
- R2: value R_Small_US -> 20
- R3: value R_Small_US -> 10K
- R4: value R_Small_US -> 200
- R5: value R_Small_US -> 4.7K
- R6: value R_Small_US -> 1K
- R8: value R_Small_US -> 3.6K
Connections:
- net GPIO0 renamed LCD_EN
- net GPIO1 renamed LCD_RS
- net GPIO2 renamed LCD_D0
- net GPIO3 renamed LCD_D1
- net GPIO4 renamed LCD_D2
- net GPIO5 renamed LCD_D3
- net GPIO6 renamed GP_RELAY
- net GPIO7 renamed SEN_TEMP
Other:
- moved on the sheet: R4

Commit message: add modification
Connections:
- net LCD_D0: now also U1.20 (PD3); no longer U1.19 (PD2)
- net LCD_D1: now also U1.19 (PD2); no longer U1.20 (PD3)
- net LCD_EN: now also U1.16 (PC6); no longer U1.15 (PC5)
- net LCD_RS: now also U1.15 (PC5); no longer U1.16 (PC6)
Changed lines of the file:
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@@
+		)
+	)
+	(label "LCD_D0"
+		(at 96.52 49.53 0)
+		(effects
+			(font
+				(size 1.27 1.27)
+			)
+			(justify left bottom)
 		)
 	)
@@
 	(label "LCD_D3"
 		(at 96.52 54.61 0)
+		(effects
+			(font
+				(size 1.27 1.27)
+			)
+			(justify left bottom)
+		)
+	)
+	(label "LCD_EN"
+		(at 40.64 59.69 0)
 		(effects
 			(font
@@
 		)
 	)
-	(label "SEN_TEMP"
-		(at 40.64 54.61 0)
+	(label "LCD_D1"
+		(at 96.52 46.99 0)
 		(effects
 			(font
@@
 		)
 	)
-	(label "LCD_D0"
-		(at 96.52 46.99 0)
+	(label "SEN_TEMP"
+		(at 40.64 54.61 0)
 		(effects
 			(font
@@
 		)
 	)
-	(label "LCD_RS"
-		(at 40.64 59.69 0)
-		(effects
-			(font
-				(size 1.27 1.27)
-			)
-			(justify left bottom)
-		)
-	)
 	(label "LCD_D2"
 		(at 203.2 67.31 0)
-		(effects
-			(font
-				(size 1.27 1.27)
-			)
-			(justify left bottom)
-		)
-	)
-	(label "LCD_D1"
-		(at 96.52 49.53 0)
 		(effects
 			(font
@@
 		)
 	)
-	(label "LCD_EN"
+	(label "LCD_RS"
 		(at 40.64 57.15 0)
 		(effects
